Commit message: Update files

File: urdf/simplearm.urdf (robot description, URDF)
Before this commit: robot simplearm, 4 links, 3 joints
Links:
- removed link simplearm_link1
- removed link simplearm_link2
- removed link simplearm_link_base
- added link link0; visual cylinder length=0.10 radius=0.10
- added link link1; visual box size=0.50 0.10 0.05
- added link link2; visual box size=0.50 0.10 0.05
Joints:
- removed joint base_link_to_simplearm_link_base
- removed joint simplearm_joint1
- removed joint simplearm_joint2
- added joint base_link_to_link0: type fixed, parent base_link, child link0, origin xyz=0 0 0.05 rpy=0 0 0
- added joint joint1: type continuous, parent link0, child link1, origin xyz=0 0 0.075 rpy=0 0 0, axis 0 0 1
- added joint joint2: type continuous, parent link1, child link2, origin xyz=0.50 0 0.05 rpy=0 0 0, axis 0 0 1
